File: slrm/slrm.kicad_pcb (KiCad board)
At the start: 4 copper layers, 82.1 x 22.5 mm, 19 parts, among them J1 Conn_01x08_Male, J2 D6, J3 D5, J4 D4, J5 D3, J6 D2, J7 D1, J8 Conn_01x08_Male, U1 74HCT04, U2 74HCT574, U3 IS62C256AL-45ULI

Commit message: final tweaks
Parts:
- renumbered J7 to D1, J6 to D2, J5 to D3, J4 to D4, J3 to D5, J2 to D6, U1 to INV, U2 to LATCH, U3 to SRAM
Other:
- board text added: "github.com/derekfountain/zx-spectrum-lower-ram v1.0"
Changed lines of the file:
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@@
     (property "Sheetname" "")
     (attr through_hole)
-    (fp_text reference "J2" (at 0 -2.06) (layer "F.SilkS")
+    (fp_text reference "D6" (at 2.68 -0.03) (layer "F.SilkS")
       (effects (font (size 1 1) (thickness 0.15)))
     )
@@
     (property "Sheetname" "")
     (attr through_hole)
-    (fp_text reference "J6" (at 0 -2.06) (layer "F.SilkS")
+    (fp_text reference "D2" (at 0 -2.06) (layer "F.SilkS")
       (effects (font (size 1 1) (thickness 0.15)))
     )
@@
     (property "Sheetname" "")
     (attr through_hole)
-    (fp_text reference "J4" (at 0 -2.06) (layer "F.SilkS")
+    (fp_text reference "D4" (at 2.65 0.03) (layer "F.SilkS")
       (effects (font (size 1 1) (thickness 0.15)))
     )
@@
     (property "Sheetname" "")
     (attr through_hole)
-    (fp_text reference "U3" (at 0 10.281191 90) (layer "F.SilkS")
+    (fp_text reference "SRAM" (at 0 10.281191 90) (layer "F.SilkS")
       (effects (font (size 1.00137 1.00137) (thickness 0.15)))
     )
@@
     (property "Sheetname" "")
     (attr through_hole)
-    (fp_text reference "J3" (at 0 -2.06) (layer "F.SilkS")
+    (fp_text reference "D5" (at 2.6 -0.01) (layer "F.SilkS")
       (effects (font (size 1 1) (thickness 0.15)))
     )
@@
     (property "Sheetname" "")
     (attr through_hole)
-    (fp_text reference "J7" (at 0 -2.06) (layer "F.SilkS")
+    (fp_text reference "D1" (at 0 -2.06) (layer "F.SilkS")
       (effects (font (size 1 1) (thickness 0.15)))
     )
@@
     (property "Sheetname" "")
     (attr smd)
-    (fp_text reference "U2" (at 0 -7.35 90) (layer "F.SilkS")
+    (fp_text reference "LATCH" (at -6.98 -0.07) (layer "F.SilkS")
       (effects (font (size 1 1) (thickness 0.15)))
     )
@@
     (property "Sheetname" "")
     (attr smd)
-    (fp_text reference "U1" (at 0 5.475 90) (layer "F.SilkS")
+    (fp_text reference "INV" (at -1.77 -5.775) (layer "F.SilkS")
       (effects (font (size 1 1) (thickness 0.15)))
     )
@@
     (property "Sheetname" "")
     (attr through_hole)
-    (fp_text reference "J5" (at 0 -2.06) (layer "F.SilkS")
+    (fp_text reference "D3" (at 0 -2.06) (layer "F.SilkS")
       (effects (font (size 1 1) (thickness 0.15)))
     )
@@
       (net 17 "ZX_WRITE"))
   )
+  (gr_circle (center 135.04 93.32) (end 135.14 93.32) (layer "F.SilkS") (width 0.15) (fill none))
+  (gr_circle (center 176.48 96.82) (end 176.58 96.82) (layer "F.SilkS") (width 0.15) (fill none))
   (gr_rect locked (start 108.735694 83.921454) (end 190.788015 106.408096) (layer "Edge.Cuts") (width 0.1) (fill none))
+  (gr_text "github.com/derekfountain/zx-spectrum-lower-ram v1.0" (at 169.59 85.13) (layer "F.SilkS")
+    (effects (font (size 1 0.5) (thickness 0.125)))
+  )
   (segment (start 133.815 103.69) (end 133.89 103.69) (width 0.35) (layer "F.Cu") (net 1))
   (segment (start 176.725 103.475) (end 179 103.475) (width 0.35) (layer "F.Cu") (net 1))
@@
   (via (at 176.7 103.5) (size 0.8) (drill 0.4) (layers "F.Cu" "B.Cu") (net 1))
   (via (at 140.35 92.65) (size 0.8) (drill 0.4) (layers "F.Cu" "B.Cu") (net 1))
+  (segment (start 141.903809 104.14) (end 140.56 104.14) (width 0.35) (layer "F.Cu") (net 2))
   (segment (start 136.3 96.875) (end 136.3 101.2) (width 0.35) (layer "F.Cu") (net 2))
   (segment (start 140.5 104.2) (end 140.5 100.339583) (width 0.35) (layer "F.Cu") (net 2))
@@
   (segment (start 171.9 100.2) (end 169.8 100.2) (width 0.35) (layer "F.Cu") (net 2))
   (segment (start 135.49 94.39) (end 135.5 94.4) (width 0.35) (layer "F.Cu") (net 2))
-  (segment (start 142.493809 103.55) (end 141.15 103.55) (width 0.35) (layer "F.Cu") (net 2))
   (segment (start 174.015 102.665) (end 174.015 100.815) (width 0.35) (layer "F.Cu") (net 2))
-  (segment (start 141.15 103.55) (end 140.5 104.2) (width 0.35) (layer "F.Cu") (net 2))
   (segment (start 140.5 100.339583) (end 139.9 99.739583) (width 0.35) (layer "F.Cu") (net 2))
   (segment (start 133.815 94.39) (end 135.49 94.39) (width 0.35) (layer "F.Cu") (net 2))
@@
   (segment (start 172.745 97.715) (end 172.745 99.455) (width 0.35) (layer "F.Cu") (net 2))
   (segment (start 169.8 100.2) (end 167.6 100.2) (width 0.35) (layer "F.Cu") (net 2))
+  (segment (start 142.493809 103.55) (end 141.903809 104.14) (width 0.35) (layer "F.Cu") (net 2))
   (segment (start 171.475 102.665) (end 171.475 100.625) (width 0.35) (layer "F.Cu") (net 2))
+  (segment (start 140.56 104.14) (end 140.5 104.2) (width 0.35) (layer "F.Cu") (net 2))
   (segment (start 122.385 93.415) (end 123 92.8) (width 0.35) (layer "F.Cu") (net 2))
   (segment (start 123.655 93.455) (end 123 92.8) (width 0.35) (layer "F.Cu") (net 2))

Commit message: v1.0, fab files sent off
Routing:
- net GND: track 45.1 -> 44.4 mm
Changed lines of the file:
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@@
       (layerselection 0x00010fc_ffffffff)
       (disableapertmacros false)
-      (usegerberextensions false)
-      (usegerberattributes true)
+      (usegerberextensions true)
+      (usegerberattributes false)
       (usegerberadvancedattributes true)
-      (creategerberjobfile true)
+      (creategerberjobfile false)
       (svguseinch false)
       (svgprecision 6)
@@
       (plotinvisibletext false)
       (sketchpadsonfab false)
-      (subtractmaskfromsilk false)
+      (subtractmaskfromsilk true)
       (outputformat 1)
       (mirror false)
-      (drillshape 1)
+      (drillshape 0)
       (scaleselection 1)
-      (outputdirectory "")
+      (outputdirectory "fab1.0")
     )
   )
@@
     (fp_line (start -1.6 -0.8) (end 1.6 -0.8) (layer "F.Fab") (width 0.1))
     (fp_line (start 1.6 -0.8) (end 1.6 0.8) (layer "F.Fab") (width 0.1))
-    (pad "1" smd roundrect locked (at -1.475 0 90) (size 1.15 1.8) (layers "F.Cu" "F.Paste" "F.Mask") (roundrect_rratio 0.217391)
+    (pad "1" smd roundrect locked (at -1.475 0 90) (size 1.15 1.8) (layers "F.Cu" "F.Paste" "F.Mask") (roundrect_rratio 0.2173913043)
       (net 1 "+5V") (pintype "passive"))
-    (pad "2" smd roundrect locked (at 1.475 0 90) (size 1.15 1.8) (layers "F.Cu" "F.Paste" "F.Mask") (roundrect_rratio 0.217391)
+    (pad "2" smd roundrect locked (at 1.475 0 90) (size 1.15 1.8) (layers "F.Cu" "F.Paste" "F.Mask") (roundrect_rratio 0.2173913043)
       (net 2 "GND") (pintype "passive"))
     (model "${KICAD6_3DMODEL_DIR}/Capacitor_SMD.3dshapes/C_1206_3216Metric.wrl"
@@
     (fp_line (start 1.6 0.8) (end -1.6 0.8) (layer "F.Fab") (width 0.1))
     (fp_line (start 1.6 -0.8) (end 1.6 0.8) (layer "F.Fab") (width 0.1))
-    (pad "1" smd roundrect locked (at -1.475 0 90) (size 1.15 1.8) (layers "F.Cu" "F.Paste" "F.Mask") (roundrect_rratio 0.217391)
+    (pad "1" smd roundrect locked (at -1.475 0 90) (size 1.15 1.8) (layers "F.Cu" "F.Paste" "F.Mask") (roundrect_rratio 0.2173913043)
       (net 1 "+5V") (pintype "passive"))
-    (pad "2" smd roundrect locked (at 1.475 0 90) (size 1.15 1.8) (layers "F.Cu" "F.Paste" "F.Mask") (roundrect_rratio 0.217391)
+    (pad "2" smd roundrect locked (at 1.475 0 90) (size 1.15 1.8) (layers "F.Cu" "F.Paste" "F.Mask") (roundrect_rratio 0.2173913043)
       (net 2 "GND") (pintype "passive"))
     (model "${KICAD6_3DMODEL_DIR}/Capacitor_SMD.3dshapes/C_1206_3216Metric.wrl"
@@
     (fp_line (start -1.6 -0.8) (end 1.6 -0.8) (layer "F.Fab") (width 0.1))
     (fp_line (start -1.6 0.8) (end -1.6 -0.8) (layer "F.Fab") (width 0.1))
-    (pad "1" smd roundrect (at -1.475 0 270) (size 1.15 1.8) (layers "F.Cu" "F.Paste" "F.Mask") (roundrect_rratio 0.217391)
+    (pad "1" smd roundrect (at -1.475 0 270) (size 1.15 1.8) (layers "F.Cu" "F.Paste" "F.Mask") (roundrect_rratio 0.2173913043)
       (net 1 "+5V") (pintype "passive"))
-    (pad "2" smd roundrect (at 1.475 0 270) (size 1.15 1.8) (layers "F.Cu" "F.Paste" "F.Mask") (roundrect_rratio 0.217391)
+    (pad "2" smd roundrect (at 1.475 0 270) (size 1.15 1.8) (layers "F.Cu" "F.Paste" "F.Mask") (roundrect_rratio 0.2173913043)
       (net 2 "GND") (pintype "passive"))
     (model "${KICAD6_3DMODEL_DIR}/Capacitor_SMD.3dshapes/C_1206_3216Metric.wrl"
@@
   (segment (start 167.6 100.2) (end 167.6 97.78) (width 0.35) (layer "F.Cu") (net 2))
   (segment (start 172.745 99.455) (end 172.7 99.5) (width 0.35) (layer "F.Cu") (net 2))
+  (segment (start 135.5 94.4) (end 135.5 96.075) (width 0.35) (layer "F.Cu") (net 2))
   (segment (start 169.8 100.2) (end 170.2 99.8) (width 0.35) (layer "F.Cu") (net 2))
   (segment (start 159.003809 103.55) (end 160.45 103.55) (width 0.35) (layer "F.Cu") (net 2))
@@
   (segment (start 169.8 100.2) (end 167.6 100.2) (width 0.35) (layer "F.Cu") (net 2))
   (segment (start 142.493809 103.55) (end 141.903809 104.14) (width 0.35) (layer "F.Cu") (net 2))
+  (segment (start 135.5 96.075) (end 136.3 96.875) (width 0.35) (layer "F.Cu") (net 2))
   (segment (start 171.475 102.665) (end 171.475 100.625) (width 0.35) (layer "F.Cu") (net 2))
   (segment (start 140.56 104.14) (end 140.5 104.2) (width 0.35) (layer "F.Cu") (net 2))
   (segment (start 122.385 93.415) (end 123 92.8) (width 0.35) (layer "F.Cu") (net 2))
   (segment (start 123.655 93.455) (end 123 92.8) (width 0.35) (layer "F.Cu") (net 2))
-  (segment (start 133.815 94.39) (end 136.3 96.875) (width 0.35) (layer "F.Cu") (net 2))
   (segment (start 168.935 101.065) (end 169.8 100.2) (width 0.35) (layer "F.Cu") (net 2))
   (segment (start 171.475 100.625) (end 171.9 100.2) (width 0.35) (layer "F.Cu") (net 2))

Commit message: work towards fab2
Parts:
- added +5V: TestPoint_THTPad_D2.0mm_Drill1.0mm, TestPoint:TestPoint_THTPad_D2.0mm_Drill1.0mm, F.Cu at (187.7, 104.7)
- added ?: , , F.Cu at (111.5, 95.4)
- added ?: , , F.Cu at (187.8, 96.5)
- added ?: , , F.Cu at (111.6, 90.4)
- added C4: C_Small, Capacitor_THT:C_Disc_D4.3mm_W1.9mm_P5.00mm, F.Cu at (177.4, 85.7)
- added GND: TestPoint_THTPad_D2.0mm_Drill1.0mm, TestPoint:TestPoint_THTPad_D2.0mm_Drill1.0mm, F.Cu at (187.6, 100.7)
- added R1: 270R, Resistor_THT:R_Axial_DIN0207_L6.3mm_D2.5mm_P10.16mm_Horizontal, F.Cu at (162.6, 85.8)
- LATCH1: renamed from LATCH; footprint Package_SO:SOIC-20W_7.5x12.8mm_P1.27mm -> Package_SO:SO-20_5.3x12.6mm_P1.27mm
- ZX CAS: renamed from CAS
- moved RAS 4.04 mm to (187.9, 92.5)
- moved ZX CAS 3.22 mm to (111.6, 87.2)
- moved WR 3.08 mm to (187.8, 88.4)
- moved GND 2.94 mm to (111.5, 99.9)
- moved +5V 2.82 mm to (111.5, 104.2)
- renumbered INV to INV1, SRAM to SRAM1
Connections:
- INV1 pad 3: GND -> DELAYED_ZX_CAS
- INV1 pad 4: unconnected-(U1-Pad4) -> INV_DELAYED_ZX_CAS
- INV1 pad 5: GND -> INV_DELAYED_ZX_CAS
- INV1 pad 6: unconnected-(U1-Pad6) -> DELAYED_CAS
- SRAM1 pad 20: ZX_CAS -> DELAYED_CAS
Routing:
- net DELAYED_CAS: track 0.00 -> 66.4 mm, vias 0 -> 3
- net DELAYED_ZX_CAS: track 0.00 -> 18.7 mm
- net RAS_INV: track 58.3 -> 73.8 mm
- net GND: track 44.4 -> 31.8 mm, vias 7 -> 10
- net ZX_CAS: track 42.3 -> 53.5 mm, vias 2 -> 1
- net INV_DELAYED_ZX_CAS: track 0.00 -> 8.24 mm
- net ZX_A0: track 68.3 -> 70.5 mm
- net ZX_A6: track 34.1 -> 32.6 mm
- net ZX_A3: track 45.1 -> 43.9 mm
- net ZX_A1: track 61.3 -> 62.5 mm
- net RAS_A4: track 27.0 -> 25.8 mm
- net RAS_A3: track 27.8 -> 26.6 mm
- net RAS_A2: track 28.6 -> 27.4 mm
- net RAS_A1: track 29.0 -> 27.8 mm
- net RAS_A0: track 29.5 -> 28.3 mm
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Other:
- board text added: "A0"
- board text added: "D'CAS"
- board text added: "INV_RAS"
- board text added: "github.com/derekfountain/zx-spectrum-lower-ram v1.1"
- board text removed: "github.com/derekfountain/zx-spectrum-lower-ram v1.0"
