File: slrm/slrm.kicad_pcb (KiCad board)
At the start: 4 copper layers, 82.1 x 22.5 mm, 26 parts, among them J1 Conn_01x08_Male, J8 Conn_01x08_Male

Commit message: version 1.2 gerbers created
Parts:
- removed +5V (x2), GND (x2), RAS, WR: TestPoint_THTPad_D2.0mm_Drill1.0mm, TestPoint:TestPoint_THTPad_D2.0mm_Drill1.0mm
- removed ? (x3): , 
- removed ZX CAS: TestPoint_THTPad_D2.0mm_Drill1.0mm, TestPoint:TestPoint_THTPad_D2.0mm_Drill1.0mm
- added C4: C_Small, Capacitor_SMD:C_1206_3216Metric, F.Cu at (179.9, 88.2)
- added REF**: R_1206_3216Metric, Resistor_SMD:R_1206_3216Metric, F.Cu at (167.7, 85.8)
Routing:
- net DELAYED_CAS: track 66.4 -> 22.0 mm, vias 3 -> 2
- net RAS_INV: track 73.8 -> 58.3 mm
- net DELAYED_ZX_CAS: track 18.7 -> 25.1 mm
- net ZX_WRITE: track 48.0 -> 41.8 mm
- net ZX_RAS: track 16.9 -> 11.3 mm
- net ZX_A0: track 70.5 -> 65.6 mm
- net ZX_CAS: track 53.5 -> 48.7 mm
- net GND: track 31.8 -> 34.7 mm
Other:
- board size 82.1 x 22.5 mm -> 67.1 x 22.5 mm
- board text added: "github.com/derekfountain/zx-spectrum-lower-ram v1.2"
- board text removed: "A0"
- board text removed: "D'CAS"
- board text removed: "INV_RAS"
- board text removed: "github.com/derekfountain/zx-spectrum-lower-ram v1.1"
